File: pcb/fiberaudio-108.kicad_pcb (KiCad board)
At the start: 2 copper layers, 45 x 45 mm, 43 parts, among them J1 USB_B_Mini, J2 PLT133_T10W, Q1 SI2301CDS, SW1 MUTE, U1 AT93C46D, U2 CM108AH, U3 SRV05-4, Y1 12MHz

Commit message: Fix USBD disco at U3; Adjust VBUS/+5 routing; Update to rev.4
Parts:
- moved U3 0.10 mm to (130.0, 55.0), turned to 90 degrees
- renumbered TPe to TP8
Connections:
- R3 pad 1: /USBD_R_N -> /USBD_N
- R4 pad 1: /USBD_R_P -> /USBD_P
- U3 pad 1: /USBD_N -> Net-(U3-Pad1)
- U3 pad 3: /USBD_P -> /USBD_N
- U3 pad 4: /USBD_R_N -> /USBD_P
- U3 pad 6: /USBD_R_P -> Net-(U3-Pad6)
Routing:
- net GND: track 101.5 -> 119.2 mm, vias 34 -> 32
- net /USBD_P: track 11.0 -> 18.4 mm, vias 0 -> 2
- net +5V: track 53.7 -> 58.8 mm
- net /USBD_N: track 13.3 -> 17.6 mm
- net /USBD_R_P: track 2.00 -> 0.00 mm
- net /USBD_R_N: track 2.00 -> 0.00 mm
- net Net-(C13-Pad1): track 12.7 -> 12.0 mm
Other:
- board text added: "rev.4"

Commit message: Rev. 5; Add ALTN part for ESD diode; Adjust layout
Parts:
- J2: value PLT133_T10W -> PLT133/T10W
- moved C13 6.01 mm to (116.8, 56.0), turned to 180 degrees
- moved R1 3.95 mm to (109.2, 66.2)
- moved C9 3.26 mm to (136.2, 72.2)
- moved C11 3.02 mm to (136.2, 70.8)
- moved C12 2.85 mm to (136.2, 69.2)
- moved C3 2.00 mm to (138.0, 65.0)
- moved C7 2.00 mm to (111.0, 73.0)
- moved C4 1.50 mm to (136.5, 65.0)
- moved C8 1.25 mm to (134.5, 65.0)
- moved C1 1.06 mm to (107.8, 66.2), turned to 90 degrees
- moved Y1 1.00 mm to (114.0, 73.0)
- moved C5 0.75 mm to (133.0, 65.0)
Connections:
- U3 pad 1: Net-(U3-Pad1) -> /USBD_N
- U3 pad 3: /USBD_N -> Net-(U3-Pad3)
- U3 pad 4: /USBD_P -> Net-(U3-Pad4)
- U3 pad 6: Net-(U3-Pad6) -> /USBD_P
Routing:
- net +5V: track 58.8 -> 51.5 mm
- net GND: track 119.2 -> 112.9 mm
- net +3V3: track 60.8 -> 55.6 mm
- net Net-(C9-Pad1): track 6.79 -> 3.31 mm
- net Net-(R1-Pad2): track 6.16 -> 3.11 mm
- net /SPDIF_MOD: track 29.9 -> 27.6 mm
- net Net-(C7-Pad1): track 17.1 -> 15.2 mm
- net Net-(C13-Pad1): track 12.0 -> 10.3 mm
- net Net-(C6-Pad1): track 11.0 -> 9.38 mm
- net /USBD_P: track 18.4 -> 19.7 mm
- net /USBD_N: track 17.6 -> 16.6 mm
Other:
- board text added: "rev.5"
- board text removed: "rev.4"
